File: Shutter_RF.kicad_pcb (KiCad board)
At the start: 2 copper layers, 50 x 50 mm, 30 parts, among them J1 Mains, J10 5V, J2 Conn_01x03, J3 SYN480, J4 SYN115, J5 Conn_01x02, J6 IIC, J7 485, J8 Position, J9 Temp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

Commit message: Common Folder
Routing:
- net /A: track 55.5 -> 57.1 mm
Changed lines of the file:
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@@
-(kicad_pcb (version 20171130) (host pcbnew 5.0.2-bee76a0~70~ubuntu16.04.1)
+(kicad_pcb (version 20171130) (host pcbnew "(5.0.2)-1")
   (general
     (thickness 1.6)
     (drawings 23)
-    (tracks 334)
+    (tracks 333)
     (zones 0)
     (modules 30)
@@
     (solder_mask_min_width 0.25)
     (aux_axis_origin 0 0)
-    (visible_elements FFFDFF7F)
+    (visible_elements 7FFFFFFF)
     (pcbplotparams
       (layerselection 0x010fc_ffffffff)
@@
   (segment (start 120.015 127.889) (end 121.92 125.984) (width 0.25) (layer B.Cu) (net 15))
   (segment (start 121.92 125.984) (end 125.222 125.984) (width 0.25) (layer B.Cu) (net 15))
-  (segment (start 123.698 125.984) (end 126.111 125.984) (width 0.25) (layer B.Cu) (net 15))
-  (segment (start 126.111 125.984) (end 126.365 125.984) (width 0.25) (layer B.Cu) (net 15))
-  (segment (start 126.365 125.984) (end 127 125.349) (width 0.25) (layer B.Cu) (net 15))
-  (segment (start 128.524 125.349) (end 128.524 122.936) (width 0.25) (layer B.Cu) (net 15))
   (segment (start 109.335 113.425) (end 109.347 113.437) (width 0.25) (layer F.Cu) (net 15))
   (segment (start 109.335 112.4) (end 109.335 113.425) (width 0.25) (layer F.Cu) (net 15))
@@
   (via (at 128.524 122.936) (size 0.8) (drill 0.4) (layers F.Cu B.Cu) (net 15))
   (segment (start 128.524 120.269) (end 128.524 122.936) (width 0.25) (layer F.Cu) (net 15))
+  (segment (start 128.524 125.349) (end 128.524 122.936) (width 0.25) (layer B.Cu) (net 15))
+  (segment (start 123.698 125.984) (end 127.889 125.984) (width 0.25) (layer B.Cu) (net 15))
+  (segment (start 127.889 125.984) (end 128.524 125.349) (width 0.25) (layer B.Cu) (net 15))
   (segment (start 109.6 133.8) (end 110.744 132.656) (width 0.25) (layer F.Cu) (net 16))
   (segment (start 108.5 133.8) (end 109.6 133.8) (width 0.25) (layer F.Cu) (net 16))
@@
   (segment (start 120.015 126.111) (end 120.777 125.349) (width 0.25) (layer B.Cu) (net 16))
   (segment (start 120.777 125.349) (end 127 125.349) (width 0.25) (layer B.Cu) (net 16))
-  (segment (start 125.476 125.349) (end 125.984 124.841) (width 0.25) (layer B.Cu) (net 16))
   (segment (start 127.508 124.841) (end 127.508 123.063) (width 0.25) (layer B.Cu) (net 16))
   (via (at 127.508 123.063) (size 0.8) (drill 0.4) (layers F.Cu B.Cu) (net 16))
@@
   (segment (start 108.065 115.431) (end 108.077 115.443) (width 0.25) (layer F.Cu) (net 16))
   (segment (start 108.065 112.4) (end 108.065 115.431) (width 0.25) (layer F.Cu) (net 16))
+  (segment (start 127 125.349) (end 127.508 124.841) (width 0.25) (layer B.Cu) (net 16))
   (segment (start 117.24975 124.012331) (end 117.094 124.168081) (width 0.25) (layer F.Cu) (net 17))
   (segment (start 117.24975 122.598118) (end 117.24975 124.012331) (width 0.25) (layer F.Cu) (net 17))
